File: hardware/boards/glasgow/revD1/USB.kicad_sch (KiCad schematic)
At the start: 24 parts, among them J1 USB-C, U4 FUSB302B01MPX, U5 TPS259472ARPW

Commit message: start from 4 V, new inv bubo, more testpoints, synsyn through LS
Parts:
- removed R259: 0, Resistor_SMD:R_0402_1005Metric, symbol Device:R_Small
- added R257: 0, Resistor_SMD:R_0402_1005Metric, symbol Device:R_Small
- added TP14: VBUS, symbol Connector:TestPoint
- added TP15: CC1, symbol Connector:TestPoint
- R24: value 330k -> 280k; LCSC C25778 -> (none); MPN 0402WGF3303TCE -> (none)
Connections:
- net CC1: now also TP15.1
- net ~{INT}: now also R257.2
- net at U4.5 (INT_N): now also R257.1
- net VUSB renamed VBUS
- net VBUS: now also TP14.1
Other:
- note added: "Power good threshold = 4 V Inverting buck-boost in Power sheet needs that much to start up initially."
- note removed: "Power good threshold = 4.5V Inverting buck-boost in Power sheet needs that much to start up initially."

Commit message: wip
Parts:
- TP14, TP15: footprint (none) -> TestPoint:TestPoint_Pad_D1.0mm
Changed lines of the file:
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@@
 			)
 		)
-		(property "Footprint" ""
+		(property "Footprint" "TestPoint:TestPoint_Pad_D1.0mm"
 			(at 102.87 77.47 0)
 			(hide yes)
@@
 			)
 		)
-		(property "Footprint" ""
+		(property "Footprint" "TestPoint:TestPoint_Pad_D1.0mm"
 			(at 102.87 99.06 0)
 			(hide yes)

Commit message: update bom
Parts:
- C20: LCSC C6144275 -> C19170936; MPN CC0402KRX7R9BB132 -> C0402C132J5GACTU
- R23: LCSC C185429 -> C113479; MPN RC0402FR-072K87L -> 0402WGF2871TCE
- R24: LCSC (none) -> C2929997; MPN (none) -> FRC0402F2803TS
- R25: LCSC C25534 -> C25750; MPN 0402WGJ0124TCE -> 0402WGF1203TCE
- R257: LCSC (none) -> C851623; MPN (none) -> PE0402FRF470R05L
- TP14, TP15: now not fitted
Changed lines of the file:
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@@
 			)
 		)
-		(property "LCSC" "C25534"
+		(property "LCSC" "C25750"
 			(at 224.79 91.44 0)
 			(hide yes)
@@
 			)
 		)
-		(property "MPN" "0402WGJ0124TCE"
+		(property "MPN" "0402WGF1203TCE"
 			(at 224.79 91.44 0)
 			(hide yes)
@@
 			)
 		)
-		(property "LCSC" "C185429"
+		(property "LCSC" "C113479"
 			(at 191.77 95.25 0)
 			(hide yes)
@@
 			)
 		)
-		(property "MPN" "RC0402FR-072K87L"
+		(property "MPN" "0402WGF2871TCE"
 			(at 191.77 95.25 0)
 			(hide yes)
@@
 			)
 		)
-		(property "Datasheet" ""
+		(property "Datasheet" "https://jlc-prod-smt.oss-eu-central-1.aliyuncs.com/smtDataManualFile/8589927047016308736-C851623.pdf?response-content-disposition=attachment%3B%20filename%3DC851623.pdf%3B%20filename%2A%3DUTF-8%27%27C851623.pdf&x-oss-date=20260524T222115Z&x-oss-expires=1800&x-oss-security-token=CAISgAN1q6Ft5B2yfSjIr5rzGuj8u7FwxZWmN2fpnloTa9xgm5TBkTz2IHhMdHJsAOodtv0%2FmmhT6PkclqRLcbhpcmfjV%2BZHzLB8qZxruQFM4J7b16cNrbH4M4H6aXeirtuwDsz9SNTCALjPD3nPii50x5bjaDymRCbLGJaViJlhHLN1Ow6jdmhpCctxLAlvo9NgFxm3D%2Fu2NQPwiWf9FVdhvhEG6Vly8qOi2MaRmFy8yFTx0b0SvJ%2BjYMrmPctoN9JnSdC5mfdzau3a1TJ84gRD0a5wkaVA1zbDs5bfISEIuUzebreLqY03dV4mOvdqIcMe8qigz88fk%2FfIioH6xyxKOexoSCnFTOiiupCcQLPyao9jLu6iayqViY7QaIOTqQohZmkAMwVOasAsI3Ngh4zF97Qt0cVNkXO9gWfLI8DtuMleWgrjRep9MnSgc5lCkRRYwGs1287ugXlSQzo890KPDAEovaKCnZ2ZSfh7Y4sNknI6i%2Bfc2Se2MIkIQ%2Ff0nKKWD5sagAEVLZ0dNN6q3YOOSB9X6kKYngn4Qecl14LG8RslXmyKAL47guIqkF4EWqJOQF54WLvQKmkK5PDichoxcAz4wyY%2B9BygnI7Y0QfZa40e%2Fp8aMKghMOKl00uJRzKspcYtrccmbdf9wpWfPEGtDzOmmsxEF5ZymPzPuf5w6dfl4hk2FiAA&x-oss-signature-version=OSS4-HMAC-SHA256&x-oss-credential=STS.NYFQRHVnQrWM5AXzZFgSLtQjs%2F20260524%2Feu-central-1%2Foss%2Faliyun_v4_request&x-oss-signature=e7e5476dff298cf10706224e96472dab3addfe113fb1c452d35c5a44f90f1097"
 			(at 167.64 102.87 0)
 			(hide yes)
@@
 			)
 		)
-		(property "LCSC" ""
+		(property "LCSC" "C851623"
 			(at 167.64 102.87 0)
 			(hide yes)
@@
 			)
 		)
-		(property "MPN" ""
+		(property "MPN" "PE0402FRF470R05L"
 			(at 167.64 102.87 0)
 			(hide yes)
@@
 			)
 		)
-		(property "LCSC" ""
+		(property "LCSC" "C2929997"
 			(at 224.79 83.82 0)
 			(hide yes)
@@
 			)
 		)
-		(property "MPN" ""
+		(property "MPN" "FRC0402F2803TS"
 			(at 224.79 83.82 0)
 			(hide yes)
@@
 		(on_board yes)
 		(in_pos_files yes)
-		(dnp no)
+		(dnp yes)
 		(fields_autoplaced yes)
 		(property "Reference" "TP14"
@@
 			)
 		)
-		(property "LCSC" "C6144275"
+		(property "LCSC" "C19170936"
 			(at 214.63 92.71 0)
 			(hide yes)
@@
 			)
 		)
-		(property "MPN" "CC0402KRX7R9BB132"
+		(property "MPN" "C0402C132J5GACTU"
 			(at 214.63 92.71 0)
 			(hide yes)
@@
 		(on_board yes)
 		(in_pos_files yes)
-		(dnp no)
+		(dnp yes)
 		(fields_autoplaced yes)
 		(property "Reference" "TP15"

Commit message: misc review changes
disconnect eFuse PG and add comments in schematic as to why
add slew-rate limiting resistor to NAFE clock
add esd diode to external clock output
fix USB D+/D- diff-pairs
update schematic to current date and set revision to D1
fix RAM balls B3/B4 assignment
Parts:
- added R252: 0, Resistor_SMD:R_0402_1005Metric, symbol Device:R_Small
Connections:
- net PG: now also R252.2; no longer U5.3 (PG)
- new net: R252.1, U5.3 (PG)
Other:
- note added: "Ignore PG. We have a separate UVLO, eFuse still does its job and won't prevent ~{RESET} from going high when the board is powered by an addon instead of bus power."
- moved on the sheet: C21, C22, R24, R25
