File: hardware/boards/glasgow/revD1/io_buffer.kicad_sch (KiCad schematic)
At the start: 17 parts, among them U24 PCA6416APW, U25 PCA6416APW, U8 LFE5U-25F-8BG256x

Commit message: start from 4 V, new inv bubo, more testpoints, synsyn through LS
Parts:
- removed R257: 0, Resistor_SMD:R_0402_1005Metric, symbol Device:R_Small
- added R268: 0, symbol Device:R_Small
- R258: footprint Resistor_SMD:R_0402_1005Metric -> (none)
Connections:
- net ~{ALERT}: now also R258.1, R268.1; no longer R258.2
- net at R83.2, U25.1 (~{INT}): now also R268.2
- net at R82.2, U24.1 (~{INT}): now also R258.2; no longer R258.1
Changed lines of the file:
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@@
 	(bus
 		(pts
-			(xy 135.89 19.05) (xy 218.44 19.05)
+			(xy 135.89 19.05) (xy 222.25 19.05)
 		)
 		(stroke
@@
 	(bus
 		(pts
-			(xy 224.79 21.59) (xy 218.44 19.05)
+			(xy 224.79 21.59) (xy 222.25 19.05)
 		)
 		(stroke
@@
 	)
 	(symbol
-		(lib_id "Device:R_Small")
-		(at 153.67 111.76 270)
-		(unit 1)
-		(body_style 1)
-		(exclude_from_sim no)
-		(in_bom yes)
-		(on_board yes)
-		(in_pos_files yes)
-		(dnp yes)
-		(fields_autoplaced yes)
-		(property "Reference" "R257"
-			(at 153.67 115.57 90)
-			(show_name no)
-			(do_not_autoplace no)
-			(effects
-				(font
-					(size 1.27 1.27)
-				)
-			)
-		)
-		(property "Value" "0"
-			(at 153.67 118.11 90)
-			(show_name no)
-			(do_not_autoplace no)
-			(effects
-				(font
-					(size 1.27 1.27)
-				)
-			)
-		)
-		(property "Footprint" "Resistor_SMD:R_0402_1005Metric"
-			(at 153.67 111.76 0)
-			(hide yes)
-			(show_name no)
-			(do_not_autoplace no)
-			(effects
-				(font
-					(size 1.27 1.27)
-				)
-			)
-		)
-		(property "Datasheet" ""
-			(at 153.67 111.76 0)
-			(hide yes)
-			(show_name no)
-			(do_not_autoplace no)
-			(effects
-				(font
-					(size 1.27 1.27)
-				)
-			)
-		)
-		(property "Description" "Resistor, small symbol"
-			(at 153.67 111.76 0)
-			(hide yes)
-			(show_name no)
-			(do_not_autoplace no)
-			(effects
-				(font
-					(size 1.27 1.27)
-				)
-			)
-		)
-		(property "LCSC" ""
-			(at 153.67 111.76 0)
-			(hide yes)
-			(show_name no)
-			(do_not_autoplace no)
-			(effects
-				(font
-					(size 1.27 1.27)
-				)
-			)
-		)
-		(property "MPN" ""
-			(at 153.67 111.76 0)
-			(hide yes)
-			(show_name no)
-			(do_not_autoplace no)
-			(effects
-				(font
-					(size 1.27 1.27)
-				)
-			)
-		)
-		(property "KLC_S4.1" ""
-			(at 153.67 111.76 0)
-			(hide yes)
-			(show_name no)
-			(do_not_autoplace no)
-			(effects
-				(font
-					(size 1.27 1.27)
-				)
-			)
-		)
-		(pin "1"
-		)
-		(pin "2"
-		)
-		(instances
-			(project "glasgow"
-				(path "/87a94d88-8a34-4311-9666-80951c15f2c0/5dfc4ecd-6671-4a7f-9f56-d6fa56b3f4ee"
-					(reference "R257")
-					(unit 1)
-				)
-			)
-		)
-	)
-	(symbol
 		(lib_id "power:+3V3")
 		(at 67.31 19.05 0)
@@
 	)
 	(symbol
-		(lib_id "Device:R_Small")
-		(at 153.67 43.18 270)
-		(unit 1)
-		(body_style 1)
-		(exclude_from_sim no)
-		(in_bom yes)
-		(on_board yes)
-		(in_pos_files yes)
-		(dnp yes)
-		(fields_autoplaced yes)
-		(property "Reference" "R258"
-			(at 153.67 46.99 90)
-			(show_name no)
-			(do_not_autoplace no)
-			(effects
-				(font
-					(size 1.27 1.27)
-				)
-			)
-		)
-		(property "Value" "0"
-			(at 153.67 49.53 90)
-			(show_name no)
-			(do_not_autoplace no)
-			(effects
-				(font
-					(size 1.27 1.27)
-				)
-			)
-		)
-		(property "Footprint" "Resistor_SMD:R_0402_1005Metric"
-			(at 153.67 43.18 0)
-			(hide yes)
-			(show_name no)
-			(do_not_autoplace no)
-			(effects
-				(font
-					(size 1.27 1.27)
-				)
-			)
-		)
-		(property "Datasheet" ""
-			(at 153.67 43.18 0)
-			(hide yes)
-			(show_name no)
-			(do_not_autoplace no)
-			(effects
-				(font
-					(size 1.27 1.27)
-				)
-			)
-		)
-		(property "Description" "Resistor, small symbol"
-			(at 153.67 43.18 0)
-			(hide yes)
-			(show_name no)
-			(do_not_autoplace no)
-			(effects
-				(font
-					(size 1.27 1.27)
-				)
-			)
-		)
-		(property "LCSC" ""
-			(at 153.67 43.18 0)
-			(hide yes)
-			(show_name no)
-			(do_not_autoplace no)
-			(effects
-				(font
-					(size 1.27 1.27)
-				)
-			)
-		)
-		(property "MPN" ""
-			(at 153.67 43.18 0)
-			(hide yes)
-			(show_name no)
-			(do_not_autoplace no)
-			(effects
-				(font
-					(size 1.27 1.27)
-				)
-			)
-		)
-		(property "KLC_S4.1" ""
-			(at 153.67 43.18 0)
-			(hide yes)
-			(show_name no)
-			(do_not_autoplace no)
-			(effects
-				(font
-					(size 1.27 1.27)
-				)
-			)
-		)
-		(pin "1"
-		)
-		(pin "2"
-		)
-		(instances
-			(project "glasgow"
-				(path "/87a94d88-8a34-4311-9666-80951c15f2c0/5dfc4ecd-6671-4a7f-9f56-d6fa56b3f4ee"
-					(reference "R258")
-					(unit 1)
-				)
-			)
-		)
-	)
-	(symbol
 		(lib_id "power:+5V")
 		(at 165.1 120.65 0)
@@
 	)
 	(symbol
+		(lib_id "Device:R_Small")
+		(at 153.67 43.18 90)
+		(unit 1)
+		(body_style 1)
+		(exclude_from_sim no)
+		(in_bom yes)
+		(on_board yes)
+		(in_pos_files yes)
+		(dnp yes)
+		(fields_autoplaced yes)
+		(property "Reference" "R258"
+			(at 153.67 46.99 90)
+			(show_name no)
+			(do_not_autoplace no)
+			(effects
+				(font
+					(size 1.016 1.016)
+				)
+			)
+		)
+		(property "Value" "0"
+			(at 153.67 49.53 90)
+			(show_name no)
+			(do_not_autoplace no)
+			(effects
+				(font
+					(size 1.27 1.27)
+				)
+			)
+		)
+		(property "Footprint" ""
+			(at 153.67 43.18 0)
+			(hide yes)
+			(show_name no)
+			(do_not_autoplace no)
+			(effects
+				(font
+					(size 1.27 1.27)
+				)
+			)
+		)
+		(property "Datasheet" ""
+			(at 153.67 43.18 0)
+			(hide yes)
+			(show_name no)
+			(do_not_autoplace no)
+			(effects
+				(font
+					(size 1.27 1.27)
+				)
+			)
+		)
+		(property "Description" "Resistor, small symbol"
+			(at 153.67 43.18 0)
+			(hide yes)
+			(show_name no)
+			(do_not_autoplace no)
+			(effects
+				(font
+					(size 1.27 1.27)
+				)
+			)
+		)
+		(pin "1"
+		)
+		(pin "2"
+		)
+		(instances
+			(project "glasgow"
+				(path "/87a94d88-8a34-4311-9666-80951c15f2c0/5dfc4ecd-6671-4a7f-9f56-d6fa56b3f4ee"
+					(reference "R258")
+					(unit 1)
+				)
+			)
+		)
+	)
+	(symbol
 		(lib_id "Means Of Circuit Design:LFE5U-25F-8BG256x")
 		(at 106.68 71.12 0)
@@
 					(unit 1)
 				)
+			)
+		)
+	)
+	(symbol
+		(lib_id "Device:R_Small")
+		(at 153.67 111.76 90)
+		(unit 1)
+		(body_style 1)
+		(exclude_from_sim no)
+		(in_bom yes)
+		(on_board yes)
+		(in_pos_files yes)
+		(dnp yes)
+		(fields_autoplaced yes)
+		(property "Reference" "R268"
+			(at 153.67 115.57 90)
+			(show_name no)
+			(do_not_autoplace no)
+			(effects
+				(font
+					(size 1.016 1.016)
+				)
+			)
+		)
+		(property "Value" "0"
+			(at 153.67 118.11 90)
+			(show_name no)
+			(do_not_autoplace no)
+			(effects
+				(font
+					(size 1.27 1.27)
+				)
+			)
+		)
+		(property "Footprint" ""
+			(at 153.67 111.76 0)
+			(hide yes)
+			(show_name no)
+			(do_not_autoplace no)
+			(effects
+				(font
+					(size 1.27 1.27)
+				)
+			)
+		)
+		(property "Datasheet" ""
+			(at 153.67 111.76 0)
+			(hide yes)
+			(show_name no)
+			(do_not_autoplace no)
+			(effects
+				(font
+					(size 1.27 1.27)
+				)
+			)
+		)
+		(property "Description" "Resistor, small symbol"
+			(at 153.67 111.76 0)
+			(hide yes)
+			(show_name no)
+			(do_not_autoplace no)
+			(effects
+				(font
+					(size 1.27 1.27)
+				)
+			)
+		)
+		(pin "1"
+		)
+		(pin "2"
+		)
+		(instances
+			(project "glasgow"
+				(path "/87a94d88-8a34-4311-9666-80951c15f2c0/5dfc4ecd-6671-4a7f-9f56-d6fa56b3f4ee"
+					(reference "R268")
+					(unit 1)
+				)

Commit message: wip
Parts:
- R258, R268: footprint (none) -> Resistor_SMD:R_0402_1005Metric
Changed lines of the file:
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@@
 			)
 		)
-		(property "Footprint" ""
+		(property "Footprint" "Resistor_SMD:R_0402_1005Metric"
 			(at 153.67 43.18 0)
 			(hide yes)
@@
 			)
 		)
-		(property "Footprint" ""
+		(property "Footprint" "Resistor_SMD:R_0402_1005Metric"
 			(at 153.67 111.76 0)
 			(hide yes)

Commit message: get routed
Parts:
- removed R252, R253: 10k, Resistor_SMD:R_0402_1005Metric, symbol Device:R_Small
Connections:
- net +3V3: now also U24.3 (~{RESET}), U25.3 (~{RESET})
- net ~{ALERT}: now also R268.2; no longer R268.1
- net at R83.2, U25.1 (~{INT}): now also R268.1; no longer R268.2
Other:
- moved on the sheet: R268

Commit message: update bom
Parts:
- R258, R268: LCSC (none) -> C17168; MPN (none) -> 0402WGF0000TCE
- U24, U25: value PCA6416APW -> TCA6416APW; LCSC C2669733 -> C130203; MPN PCA6416APW,118 -> TCA6416APWR
Other:
- note added: "Potential alternative: NCA6416, PCA6416A"
- note added: "Swapped NXP with TI part for availability."
- note removed: "Potential alternative: NCA6416, PCAL6416"
Changed lines of the file:
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@@
 		)
 	)
-	(text "Potential alternative:\nNCA6416, PCAL6416"
+	(text "Potential alternative:\nNCA6416, PCA6416A"
 		(exclude_from_sim no)
 		(at 144.78 88.9 0)
@@
 		)
 	)
+	(text "Swapped NXP with TI part\nfor availability."
+		(exclude_from_sim no)
+		(at 154.94 68.58 0)
+		(effects
+			(font
+				(size 1.27 1.27)
+				(color 204 102 0 1)
+			)
+		)
+	)
 	(text "INA D: 1001111"
 		(exclude_from_sim no)
@@
 			)
 		)
-		(property "Value" "PCA6416APW"
+		(property "Value" "TCA6416APW"
 			(at 182.4833 86.36 0)
 			(show_name no)
@@
 			)
 		)
-		(property "Datasheet" "https://www.nxp.com/docs/en/data-sheet/PCAL6416A.pdf"
+		(property "Datasheet" "https://www.ti.com/lit/ds/symlink/tca6416a.pdf"
 			(at 180.34 59.69 0)
 			(hide yes)
@@
 			)
 		)
-		(property "LCSC" "C2669733"
+		(property "LCSC" "C130203"
 			(at 180.34 58.42 0)
 			(hide yes)
@@
 			)
 		)
-		(property "MPN" "PCA6416APW,118"
+		(property "MPN" "TCA6416APWR"
 			(at 180.34 58.42 0)
 			(hide yes)
@@
 			)
 		)
-		(property "Value" "PCA6416APW"
+		(property "Value" "TCA6416APW"
 			(at 182.4833 154.94 0)
 			(show_name no)
@@
 			)
 		)
-		(property "Datasheet" "https://www.nxp.com/docs/en/data-sheet/PCAL6416A.pdf"
+		(property "Datasheet" "https://www.ti.com/lit/ds/symlink/tca6416a.pdf"
 			(at 180.34 128.27 0)
 			(hide yes)
@@
 			)
 		)
-		(property "LCSC" "C2669733"
+		(property "LCSC" "C130203"
 			(at 180.34 127 0)
 			(hide yes)
@@
 			)
 		)
-		(property "MPN" "PCA6416APW,118"
+		(property "MPN" "TCA6416APWR"
 			(at 180.34 127 0)
 			(hide yes)
@@
 			)
 		)
+		(property "LCSC" "C17168"
+			(at 153.67 43.18 90)
+			(hide yes)
+			(show_name no)
+			(do_not_autoplace no)
+			(effects
+				(font
+					(size 1.27 1.27)
+				)
+			)
+		)
+		(property "MPN" "0402WGF0000TCE"
+			(at 153.67 43.18 90)
+			(hide yes)
+			(show_name no)
+			(do_not_autoplace no)
+			(effects
+				(font
+					(size 1.27 1.27)
+				)
+			)
+		)
 		(pin "1"
 		)
@@
 			(hide yes)
 			(show_name no)
+			(do_not_autoplace no)
+			(effects
+				(font
+					(size 1.27 1.27)
+				)
+			)
+		)
+		(property "LCSC" "C17168"
+			(at 153.67 111.76 90)
+			(hide yes)
+			(show_name no)
+			(do_not_autoplace no)
+			(effects
+				(font
+					(size 1.27 1.27)
+				)
+			)
+		)
+		(property "MPN" "0402WGF0000TCE"
+			(at 153.67 111.76 90)
+			(hide yes)
+			(show_name no)
