File: hardware/boards/glasgow/revD1/level_shifters.kicad_sch (KiCad schematic)
At the start: 101 parts, among them J7 P1, U26 74AXP1T45, U27 74AXP1T45, U28 TPS629203, U29 74AXP1T45, U30 74AXP1T45, U31 74AXP1T45, U32 74AXP1T45, U33 NCP456R, U34 INA233, U35 74AXP1T45, U36 74AXP1T45, U37 TLV6001DCK

Commit message: start from 4 V, new inv bubo, more testpoints, synsyn through LS
Parts:
- added R259: 10k, Resistor_SMD:R_0201_0603Metric, symbol Device:R_Small
- added TP17: VIO_EN, symbol Connector:TestPoint_Small
- added TP21: ~{ALERT}_Vio, symbol Connector:TestPoint_Small
- U26, U27, U29, U30, U31, U32, U35, U36: footprint Package_TO_SOT_SMD:SOT-363_SC-70-6 -> Package_TO_SOT_SMD:SOT-23-6
- U33: footprint Automated:WLCSP-6_1.4x1.0mm_P0.4mm -> Package_CSP:WLCSP-6_1.4x1.0mm_P0.4mm
Connections:
- net GND: now also R259.2
- net VIO_EN: now also TP17.1
- net V_{IO_OUT}: now also R259.1
- net ~{ALERT}_V_{IO}: now also TP21.1
Other:
- note added: "Output dschg."

Commit message: wip
Parts:
- TP17, TP21: footprint (none) -> TestPoint:TestPoint_Pad_D1.0mm
Changed lines of the file:
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@@
 			)
 		)
-		(property "Footprint" ""
+		(property "Footprint" "TestPoint:TestPoint_Pad_D1.0mm"
 			(at 50.8 147.32 0)
 			(hide yes)
@@
 			)
 		)
-		(property "Footprint" ""
+		(property "Footprint" "TestPoint:TestPoint_Pad_D1.0mm"
 			(at 167.64 170.18 0)
 			(hide yes)

Commit message: get routed
Parts:
- TP17, TP21: footprint TestPoint:TestPoint_Pad_D1.0mm -> Automated:TestPoint_Pad_D0.5mm
- U26, U27, U29, U30, U31, U32, U35, U36: footprint Package_TO_SOT_SMD:SOT-23-6 -> Package_TO_SOT_SMD:SOT-363_SC-70-6
- U33: footprint Package_CSP:WLCSP-6_1.4x1.0mm_P0.4mm -> Automated:WLCSP-6_1.4x1.0mm_P0.4mm
Connections:
- net ~{ALERT}_V_{IO}: no longer TP21.1
- net at D41.3, U34.3 (~{Alert}): now also TP21.1
Other:
- moved on the sheet: TP21
Changed lines of the file:
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@@
 	)
 	(junction
-		(at 162.56 173.99)
-		(diameter 0)
-		(color 0 0 0 0)
-	)
-	(junction
 		(at 82.55 73.66)
 		(diameter 0)
@@
 	)
 	(junction
+		(at 156.21 182.88)
+		(diameter 0)
+		(color 0 0 0 0)
+	)
+	(junction
 		(at 243.84 123.19)
 		(diameter 0)
@@
 	)
 	(bus_entry
+		(at 144.78 142.24)
+		(size 2.54 2.54)
+		(stroke
+			(width 0)
+			(type default)
+		)
+	)
+	(bus_entry
 		(at 194.31 29.21)
 		(size -2.54 -2.54)
@@
 		)
 	)
+	(wire
+		(pts
+			(xy 156.21 182.88) (xy 156.21 191.77)
+		)
+		(stroke
+			(width 0)
+			(type default)
+		)
+	)
 	(bus
 		(pts
@@
 	(wire
 		(pts
-			(xy 162.56 170.18) (xy 162.56 173.99)
-		)
-		(stroke
-			(width 0)
-			(type default)
-		)
-	)
-	(wire
-		(pts
 			(xy 127 69.85) (xy 127 73.66)
 		)
@@
 			)
 		)
-		(property "Footprint" "TestPoint:TestPoint_Pad_D1.0mm"
+		(property "Footprint" "Automated:TestPoint_Pad_D0.5mm"
 			(at 50.8 147.32 0)
 			(hide yes)
@@
 			)
 		)
-		(property "Footprint" "Package_TO_SOT_SMD:SOT-23-6"
+		(property "Footprint" "Package_TO_SOT_SMD:SOT-363_SC-70-6"
 			(at 35.56 55.88 0)
 			(hide yes)
@@
 			)
 		)
-		(property "Datasheet" "http://www.ti.com/lit/ds/symlink/sn74lvc1t45.pdf"
+		(property "Datasheet" "https://assets.nexperia.com/documents/data-sheet/74AXP1T45.pdf"
 			(at 12.7 60.96 0)
 			(hide yes)
@@
 			)
 		)
-		(property "Footprint" "Package_TO_SOT_SMD:SOT-23-6"
+		(property "Footprint" "Package_TO_SOT_SMD:SOT-363_SC-70-6"
 			(at 168.91 55.88 0)
 			(hide yes)
@@
 			)
 		)
-		(property "Datasheet" "http://www.ti.com/lit/ds/symlink/sn74lvc1t45.pdf"
+		(property "Datasheet" "https://assets.nexperia.com/documents/data-sheet/74AXP1T45.pdf"
 			(at 146.05 60.96 0)
 			(hide yes)
@@
 			)
 		)
-		(property "Footprint" "Package_CSP:WLCSP-6_1.4x1.0mm_P0.4mm"
+		(property "Footprint" "Automated:WLCSP-6_1.4x1.0mm_P0.4mm"
 			(at 140.97 130.81 0)
 			(hide yes)
@@
 			)
 		)
-		(property "KLC_S4.1" ""
-			(at 140.97 130.81 0)
-			(hide yes)
-			(show_name no)
-			(do_not_autoplace no)
-			(effects
-				(font
-					(size 1.27 1.27)
-				)
-			)
-		)
 		(pin "B2"
 		)
@@
 			)
 		)
-		(property "Footprint" "Package_TO_SOT_SMD:SOT-23-6"
+		(property "Footprint" "Package_TO_SOT_SMD:SOT-363_SC-70-6"
 			(at 35.56 96.52 0)
 			(hide yes)
@@
 			)
 		)
-		(property "Datasheet" "http://www.ti.com/lit/ds/symlink/sn74lvc1t45.pdf"
+		(property "Datasheet" "https://assets.nexperia.com/documents/data-sheet/74AXP1T45.pdf"
 			(at 12.7 101.6 0)
 			(hide yes)
@@
 			)
 		)
-		(property "Footprint" "Package_TO_SOT_SMD:SOT-23-6"
+		(property "Footprint" "Package_TO_SOT_SMD:SOT-363_SC-70-6"
 			(at 168.91 96.52 0)
 			(hide yes)
@@
 			)
 		)
-		(property "Datasheet" "http://www.ti.com/lit/ds/symlink/sn74lvc1t45.pdf"
+		(property "Datasheet" "https://assets.nexperia.com/documents/data-sheet/74AXP1T45.pdf"
 			(at 146.05 101.6 0)
 			(hide yes)
@@
 	(symbol
 		(lib_id "Connector:TestPoint_Small")
-		(at 162.56 170.18 0)
+		(at 156.21 191.77 0)
 		(unit 1)
 		(body_style 1)
@@
 		(fields_autoplaced yes)
 		(property "Reference" "TP21"
-			(at 163.83 168.9099 0)
+			(at 154.94 190.4999 0)
 			(show_name no)
 			(do_not_autoplace no)
@@
 					(size 1.27 1.27)
 				)
-				(justify left)
+				(justify right)
 			)
 		)
 		(property "Value" "~{ALERT}_Vio"
-			(at 163.83 171.4499 0)
+			(at 154.94 193.0399 0)
 			(show_name no)
 			(do_not_autoplace no)
@@
 					(size 1.27 1.27)
 				)
-				(justify left)
+				(justify right)
 			)
 		)
-		(property "Footprint" "TestPoint:TestPoint_Pad_D1.0mm"
-			(at 167.64 170.18 0)
+		(property "Footprint" "Automated:TestPoint_Pad_D0.5mm"
+			(at 161.29 191.77 0)
 			(hide yes)
 			(show_name no)
@@
 		)
 		(property "Datasheet" ""
-			(at 167.64 170.18 0)
+			(at 161.29 191.77 0)
 			(hide yes)
 			(show_name no)
@@
 		)
 		(property "Description" "test point"
-			(at 162.56 170.18 0)
+			(at 156.21 191.77 0)
 			(hide yes)
 			(show_name no)
@@
 			)
 		)
-		(property "Footprint" "Package_TO_SOT_SMD:SOT-23-6"
+		(property "Footprint" "Package_TO_SOT_SMD:SOT-363_SC-70-6"
 			(at 124.46 55.88 0)
 			(hide yes)
@@
 			)
 		)
-		(property "Datasheet" "http://www.ti.com/lit/ds/symlink/sn74lvc1t45.pdf"
+		(property "Datasheet" "https://assets.nexperia.com/documents/data-sheet/74AXP1T45.pdf"
 			(at 101.6 60.96 0)
 			(hide yes)
@@
 			)
 		)
-		(property "Footprint" "Package_TO_SOT_SMD:SOT-23-6"
+		(property "Footprint" "Package_TO_SOT_SMD:SOT-363_SC-70-6"
 			(at 80.01 96.52 0)
 			(hide yes)
@@
 			)
 		)
-		(property "Datasheet" "http://www.ti.com/lit/ds/symlink/sn74lvc1t45.pdf"
+		(property "Datasheet" "https://assets.nexperia.com/documents/data-sheet/74AXP1T45.pdf"
 			(at 57.15 101.6 0)
 			(hide yes)
@@
 			)
 		)
-		(property "Footprint" "Package_TO_SOT_SMD:SOT-23-6"
+		(property "Footprint" "Package_TO_SOT_SMD:SOT-363_SC-70-6"
 			(at 124.46 96.52 0)
 			(hide yes)
@@
 			)
 		)
-		(property "Datasheet" "http://www.ti.com/lit/ds/symlink/sn74lvc1t45.pdf"
+		(property "Datasheet" "https://assets.nexperia.com/documents/data-sheet/74AXP1T45.pdf"
 			(at 101.6 101.6 0)
 			(hide yes)
@@
 			)
 		)
-		(property "Footprint" "Package_TO_SOT_SMD:SOT-23-6"
+		(property "Footprint" "Package_TO_SOT_SMD:SOT-363_SC-70-6"
 			(at 80.01 55.88 0)
 			(hide yes)
@@
 			)
 		)
-		(property "Datasheet" "http://www.ti.com/lit/ds/symlink/sn74lvc1t45.pdf"
+		(property "Datasheet" "https://assets.nexperia.com/documents/data-sheet/74AXP1T45.pdf"
 			(at 57.15 60.96 0)
 			(hide yes)

Commit message: update bom
Parts:
- R259: LCSC (none) -> C106225; MPN (none) -> RC0201FR-0710KL
- R88: LCSC C25769 -> C1152; MPN 0402WGF2402TCE -> RC-02K243JT
- R92: value 0R -> 0; LCSC (none) -> C17168; MPN (none) -> 0402WGF0000TCE
- TP17, TP21: now not fitted
Changed lines of the file:
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@@
 		(on_board yes)
 		(in_pos_files yes)
-		(dnp no)
+		(dnp yes)
 		(fields_autoplaced yes)
 		(property "Reference" "TP17"
@@
 		(on_board yes)
 		(in_pos_files yes)
-		(dnp no)
+		(dnp yes)
 		(fields_autoplaced yes)
 		(property "Reference" "TP21"
@@
 			)
 		)
-		(property "Value" "0R"
+		(property "Value" "0"
 			(at 140.97 114.3 90)
 			(show_name no)
@@
 			)
 		)
+		(property "LCSC" "C17168"
+			(at 140.97 116.84 90)
+			(hide yes)
+			(show_name no)
+			(do_not_autoplace no)
+			(effects
+				(font
+					(size 1.27 1.27)
+				)
+			)
+		)
+		(property "MPN" "0402WGF0000TCE"
+			(at 140.97 116.84 90)
+			(hide yes)
+			(show_name no)
+			(do_not_autoplace no)
+			(effects
+				(font
+					(size 1.27 1.27)
+				)
+			)
+		)
 		(pin "2"
 		)
@@
 			)
 		)
-		(property "LCSC" "C25769"
+		(property "LCSC" "C1152"
 			(at 81.28 165.1 0)
 			(hide yes)
@@
 			)
 		)
-		(property "MPN" "0402WGF2402TCE"
+		(property "MPN" "RC-02K243JT"
 			(at 81.28 165.1 0)
 			(hide yes)
@@
 			(at 153.67 116.84 90)
 			(hide yes)
+			(show_name no)
+			(do_not_autoplace no)
+			(effects
+				(font
+					(size 1.27 1.27)
+				)
+			)
+		)
+		(property "LCSC" "C106225"
+			(at 153.67 116.84 90)
+			(hide yes)
+			(show_name no)
+			(do_not_autoplace no)
+			(effects
+				(font
+					(size 1.27 1.27)
+				)
+			)
+		)
+		(property "MPN" "RC0201FR-0710KL"
+			(at 153.67 116.84 90)
+			(hide yes)
