File: hardware/boards/glasgow/revD1/power.kicad_sch (KiCad schematic)
At the start: 101 parts, among them Q1 AO3401, Q2 AO3400, SW1 RST, U13 TLV62569PDRL, U14 TLV62569PDRL, U15 TLV61070ADBV, U16 APX811-40UG-7, U17 TLV77525DRL, U18 TLV62569PDRL, U19 TPS7A2033, U20 TPS22917DBV, U21 DAC43204, U22 SY8301, U23 SY7208CABC

Commit message: start from 4 V, new inv bubo, more testpoints, synsyn through LS
Parts:
- U21: footprint Package_DFN_QFN:WQFN-16-1EP_3x3mm_P0.5mm_EP1.68x1.68mm -> Package_DFN_QFN:WQFN-16-1EP_3x3mm_P0.5mm_EP1.68x1.68mm_ThermalVias
- U22: value SY8301 -> LMR54406; LCSC C2927130 -> C5219316; MPN SY8301ABC -> LMR54406DBVR
Connections:
- net at U20.5 (QOD): no longer R72.1
Other:
- note added: "Buck regulator in inverting buck-boost configuration. Vin min = 4 V"
- note removed: "Buck regulator in inverting buck-boost configuration."
Changed lines of the file:
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@@
 		)
 	)
-	(text "Buck regulator in inverting\nbuck-boost configuration."
+	(text "Buck regulator in inverting\nbuck-boost configuration.\nVin min = 4 V"
 		(exclude_from_sim no)
-		(at 168.91 132.08 0)
+		(at 168.91 132.715 0)
 		(effects
 			(font
@@
 			)
 		)
-		(property "Footprint" "Package_DFN_QFN:WQFN-16-1EP_3x3mm_P0.5mm_EP1.68x1.68mm"
+		(property "Footprint" "Package_DFN_QFN:WQFN-16-1EP_3x3mm_P0.5mm_EP1.68x1.68mm_ThermalVias"
 			(at 195.58 38.1 0)
 			(hide yes)
@@
 			)
 		)
-		(property "Datasheet" "https://www.lcsc.com/datasheet/C23380893.pdf"
+		(property "Datasheet" "http://www.ti.com/lit/ds/symlink/tlv755p.pdf"
 			(at 113.03 113.03 0)
 			(hide yes)
@@
 			)
 		)
-		(property "Datasheet" "www.ti.com/lit/ds/symlink/tps7a20.pdf"
+		(property "Datasheet" "http://www.ti.com/lit/ds/symlink/tps763.pdf"
 			(at 147.32 179.07 0)
 			(hide yes)
@@
 			)
 		)
-		(property "Description" "Low power 300mA LDO 3.3V fixed output voltage, SOT-23-5"
+		(property "Description" "Low power 150mA LDO 3.3V fixed output voltage, SOT-23-5"
 			(at 147.32 179.07 0)
 			(hide yes)
@@
 	)
 	(symbol
+		(lib_id "Means Of Circuit Design:SY8201")
+		(at 200.66 134.62 0)
+		(unit 1)
+		(body_style 1)
+		(exclude_from_sim no)
+		(in_bom yes)
+		(on_board yes)
+		(in_pos_files yes)
+		(dnp no)
+		(fields_autoplaced yes)
+		(property "Reference" "U22"
+			(at 200.66 129.54 0)
+			(show_name no)
+			(do_not_autoplace no)
+			(effects
+				(font
+					(size 1.27 1.27)
+				)
+			)
+		)
+		(property "Value" "LMR54406"
+			(at 200.66 132.08 0)
+			(show_name no)
+			(do_not_autoplace no)
+			(effects
+				(font
+					(size 1.27 1.27)
+				)
+			)
+		)
+		(property "Footprint" "Package_TO_SOT_SMD:SOT-23-6"
+			(at 201.93 155.956 0)
+			(hide yes)
+			(show_name no)
+			(do_not_autoplace no)
+			(effects
+				(font
+					(size 1.27 1.27)
+				)
+			)
+		)
+		(property "Datasheet" "https://www.ti.com/lit/ds/symlink/lmr54406.pdf"
+			(at 200.406 157.988 0)
+			(hide yes)
+			(show_name no)
+			(do_not_autoplace no)
+			(effects
+				(font
+					(size 1.27 1.27)
+				)
+			)
+		)
+		(property "Description" "High Efficiency Fast Response, 0.6A, 45V Input Synchronous Step Down Regulator"
+			(at 207.518 154.686 0)
+			(hide yes)
+			(show_name no)
+			(do_not_autoplace no)
+			(effects
+				(font
+					(size 1.27 1.27)
+				)
+			)
+		)
+		(property "MPN" "LMR54406DBVR"
+			(at 200.66 134.62 0)
+			(hide yes)
+			(show_name no)
+			(do_not_autoplace no)
+			(effects
+				(font
+					(size 1.27 1.27)
+				)
+			)
+		)
+		(property "LCSC" "C5219316"
+			(at 200.66 134.62 0)
+			(hide yes)
+			(show_name no)
+			(do_not_autoplace no)
+			(effects
+				(font
+					(size 1.27 1.27)
+				)
+			)
+		)
+		(pin "4"
+		)
+		(pin "1"
+		)
+		(pin "3"
+		)
+		(pin "5"
+		)
+		(pin "2"
+		)
+		(pin "6"
+		)
+		(instances
+			(project "glasgow"
+				(path "/87a94d88-8a34-4311-9666-80951c15f2c0/5e58c40f-4fbc-48ee-9161-18e9ce40e918"
+					(reference "U22")
+					(unit 1)
+				)
+			)
+		)
+	)
+	(symbol
 		(lib_id "power:+3.3V")
 		(at 74.93 173.99 0)
@@
 			)
 		)
-		(property "Datasheet" "https://www.lcsc.com/datasheet/C18207544.pdf"
+		(property "Datasheet" "https://assets.nexperia.com/documents/data-sheet/BAT54W_SER.pdf"
 			(at 81.28 169.418 0)
 			(hide yes)
@@
 	)
 	(symbol
-		(lib_id "Means Of Circuit Design:SY8201")
-		(at 200.66 134.62 0)
-		(unit 1)
-		(body_style 1)
-		(exclude_from_sim no)
-		(in_bom yes)
-		(on_board yes)
-		(in_pos_files yes)
-		(dnp no)
-		(fields_autoplaced yes)
-		(property "Reference" "U22"
-			(at 200.66 129.54 0)
-			(show_name no)
-			(do_not_autoplace no)
-			(effects
-				(font
-					(size 1.27 1.27)
-				)
-			)
-		)
-		(property "Value" "SY8301"
-			(at 200.66 132.08 0)
-			(show_name no)
-			(do_not_autoplace no)
-			(effects
-				(font
-					(size 1.27 1.27)
-				)
-			)
-		)
-		(property "Footprint" "Package_TO_SOT_SMD:SOT-23-6"
-			(at 201.93 155.956 0)
-			(hide yes)
-			(show_name no)
-			(do_not_autoplace no)
-			(effects
-				(font
-					(size 1.27 1.27)
-				)
-			)
-		)
-		(property "Datasheet" "https://www.lcsc.com/datasheet/C2927130.pdf"
-			(at 200.406 157.988 0)
-			(hide yes)
-			(show_name no)
-			(do_not_autoplace no)
-			(effects
-				(font
-					(size 1.27 1.27)
-				)
-			)
-		)
-		(property "Description" "High Efficiency Fast Response, 1A, 27V Input Synchronous Step Down Regulator"
-			(at 207.518 154.686 0)
-			(hide yes)
-			(show_name no)
-			(do_not_autoplace no)
-			(effects
-				(font
-					(size 1.27 1.27)
-				)
-			)
-		)
-		(property "MPN" "SY8301ABC"
-			(at 200.66 134.62 0)
-			(hide yes)
-			(show_name no)
-			(do_not_autoplace no)
-			(effects
-				(font
-					(size 1.27 1.27)
-				)
-			)
-		)
-		(property "LCSC" "C2927130"
-			(at 200.66 134.62 0)
-			(hide yes)
-			(show_name no)
-			(do_not_autoplace no)
-			(effects
-				(font
-					(size 1.27 1.27)
-				)
-			)
-		)
-		(property "KLC_S4.1" ""
-			(at 200.66 134.62 0)
-			(hide yes)
-			(show_name no)
-			(do_not_autoplace no)
-			(effects
-				(font
-					(size 1.27 1.27)
-				)
-			)
-		)
-		(pin "4"
-		)
-		(pin "1"
-		)
-		(pin "3"
-		)
-		(pin "5"
-		)
-		(pin "2"
-		)
-		(pin "6"
-		)
-		(instances
-			(project "glasgow"
-				(path "/87a94d88-8a34-4311-9666-80951c15f2c0/5e58c40f-4fbc-48ee-9161-18e9ce40e918"
-					(reference "U22")
-					(unit 1)
-				)
-			)
-		)
-	)
-	(symbol
 		(lib_id "Power_Supervisor:CAT811JTBI-GT3")
 		(at 49.53 158.75 0)
@@
 			)
 		)
-		(property "Datasheet" "https://www.diodes.com/datasheet/download/APX811.pdf"
+		(property "Datasheet" "http://www.onsemi.com/pub/Collateral/CAT811-D.PDF"
 			(at 40.64 176.53 0)
 			(hide yes)
@@
 			)
 		)
-		(property "Datasheet" "https://www.lcsc.com/datasheet/C178234.pdf"
+		(property "Datasheet" "https://datasheet.lcsc.com/szlcsc/Silergy-Corp-SY7208CABC_C178234.pdf"
 			(at 212.09 97.79 0)
 			(hide yes)

Commit message: get routed
Parts:
- U21: footprint Package_DFN_QFN:WQFN-16-1EP_3x3mm_P0.5mm_EP1.68x1.68mm_ThermalVias -> Package_DFN_QFN:WQFN-16-1EP_3x3mm_P0.5mm_EP1.68x1.68mm
Connections:
- net at U20.5 (QOD): now also R72.1
- net ~{FPGA_RESET} renamed FPGA_~{RESET}
Other:
- note added: "PG_{VBUS} UVLO is after the eFuse so that even if the device is powered externally it should still power up correctly."
- moved on the sheet: R72
Changed lines of the file:
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@@
 		)
 	)
+	(text "PG_{VBUS} UVLO is after the eFuse\nso that even if the device is\npowered externally it should still\npower up correctly."
+		(exclude_from_sim no)
+		(at 15.875 163.83 0)
+		(effects
+			(font
+				(size 0.635 0.635)
+			)
+			(justify left)
+		)
+	)
 	(text "Test w/o U16, should work"
 		(exclude_from_sim no)
@@
 	(wire
 		(pts
-			(xy 163.83 26.67) (xy 163.83 25.4)
+			(xy 163.83 29.21) (xy 163.83 26.67)
 		)
 		(stroke
@@
 	(wire
 		(pts
-			(xy 160.02 26.67) (xy 163.83 26.67)
+			(xy 160.02 29.21) (xy 163.83 29.21)
 		)
 		(stroke
@@
 	(wire
 		(pts
-			(xy 163.83 17.78) (xy 163.83 20.32)
+			(xy 163.83 17.78) (xy 163.83 21.59)
 		)
 		(stroke
@@
 		)
 	)
-	(hierarchical_label "~{FPGA_RESET}"
+	(hierarchical_label "FPGA_~{RESET}"
 		(shape input)
 		(at 139.7 29.21 180)
@@
 		(in_pos_files yes)
 		(dnp no)
+		(fields_autoplaced yes)
 		(property "Reference" "R59"
-			(at 26.67 153.6699 0)
+			(at 31.75 153.6699 0)
 			(show_name no)
 			(do_not_autoplace no)
@@
 					(size 1.27 1.27)
 				)
-				(justify left)
+				(justify right)
 			)
 		)
 		(property "Value" "100k"
-			(at 26.67 156.2099 0)
+			(at 31.75 156.2099 0)
 			(show_name no)
 			(do_not_autoplace no)
@@
 					(size 1.27 1.27)
 				)
-				(justify left)
+				(justify right)
 			)
 		)
@@
 			)
 		)
-		(property "Footprint" "Package_DFN_QFN:WQFN-16-1EP_3x3mm_P0.5mm_EP1.68x1.68mm_ThermalVias"
+		(property "Footprint" "Package_DFN_QFN:WQFN-16-1EP_3x3mm_P0.5mm_EP1.68x1.68mm"
 			(at 195.58 38.1 0)
 			(hide yes)
@@
 		)
 		(property "Value" "GND"
-			(at 36.83 152.3999 0)
+			(at 41.91 152.3999 0)
+			(hide yes)
 			(show_name no)
 			(do_not_autoplace no)
@@
 					(size 1.27 1.27)
 				)
-				(justify right)
+				(justify left)
 			)
 		)
@@
 	(symbol
 		(lib_id "Device:R_Small")
-		(at 163.83 22.86 180)
+		(at 163.83 24.13 180)
 		(unit 1)
 		(body_style 1)
@@
 		(fields_autoplaced yes)
 		(property "Reference" "R72"
-			(at 166.37 21.5899 0)
+			(at 166.37 22.8599 0)
 			(show_name no)
 			(do_not_autoplace no)
@@
 		)
 		(property "Value" "4.7"
-			(at 166.37 24.1299 0)
+			(at 166.37 25.3999 0)
 			(show_name no)
 			(do_not_autoplace no)
@@
 		)
 		(property "Footprint" "Resistor_SMD:R_0402_1005Metric"
-			(at 163.83 22.86 0)
+			(at 163.83 24.13 0)
 			(hide yes)
 			(show_name no)
@@
 		)
 		(property "Datasheet" ""
-			(at 163.83 22.86 0)
+			(at 163.83 24.13 0)
 			(hide yes)
 			(show_name no)
@@
 		)
 		(property "Description" "Resistor, small symbol"
-			(at 163.83 22.86 0)
+			(at 163.83 24.13 0)
 			(hide yes)
 			(show_name no)
@@
 		)
 		(property "LCSC" "C25169"
-			(at 163.83 22.86 0)
+			(at 163.83 24.13 0)
 			(hide yes)
 			(show_name no)
@@
 		)
 		(property "MPN" "0402WGJ047JTCE"
-			(at 163.83 22.86 0)
+			(at 163.83 24.13 0)
 			(hide yes)
 			(show_name no)
@@
 		)
 		(property "KLC_S4.1" ""
-			(at 163.83 22.86 0)
+			(at 163.83 24.13 0)
 			(hide yes)
 			(show_name no)

Commit message: update bom
Parts:
- R60: value 0R -> 0; LCSC (none) -> C17168; MPN (none) -> 0402WGF0000TCE
- U14, U18: MPN TLV62569PDRL -> TLV62569PDRLR
Changed lines of the file:
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@@
 			)
 		)
-		(property "Value" "0R"
+		(property "Value" "0"
 			(at 31.75 134.62 90)
 			(show_name no)
@@
 			)
 		)
+		(property "LCSC" "C17168"
+			(at 31.75 137.16 90)
+			(hide yes)
+			(show_name no)
+			(do_not_autoplace no)
+			(effects
+				(font
+					(size 1.27 1.27)
+				)
+			)
+		)
+		(property "MPN" "0402WGF0000TCE"
+			(at 31.75 137.16 90)
+			(hide yes)
+			(show_name no)
+			(do_not_autoplace no)
+			(effects
+				(font
+					(size 1.27 1.27)
+				)
+			)
+		)
 		(pin "2"
 		)
@@
 			)
 		)
-		(property "MPN" "TLV62569PDRL"
+		(property "MPN" "TLV62569PDRLR"
 			(at 114.3 82.55 0)
 			(hide yes)
@@
 			)
 		)
-		(property "MPN" "TLV62569PDRL"
+		(property "MPN" "TLV62569PDRLR"
 			(at 44.45 114.3 0)
 			(hide yes)

Commit message: misc review changes
disconnect eFuse PG and add comments in schematic as to why
add slew-rate limiting resistor to NAFE clock
add esd diode to external clock output
fix USB D+/D- diff-pairs
update schematic to current date and set revision to D1
fix RAM balls B3/B4 assignment
Other:
- note added: "PG_{VBUS} needs bus power to start up and does not set PG high even if the 5V rail is stable but bus voltage is not present."
- note removed: "PG_{VBUS} UVLO is after the eFuse so that even if the device is powered externally it should still power up correctly."
Changed lines of the file:
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@@
 	(title_block
 		(title "Power Supplies")
-		(date "2026-05-26")
-		(rev "D0")
+		(date "2026-09-22")
+		(rev "D1")
 		(company "ln / Fully Automated")
 		(comment 1 "Glasgow Debug Tool")
@@
 		)
 	)
-	(text "PG_{VBUS} UVLO is after the eFuse\nso that even if the device is\npowered externally it should still\npower up correctly."
+	(text "PG_{VBUS} needs bus power to\nstart up and does not set PG\nhigh even if the 5V rail is\nstable but bus voltage is not\npresent."
 		(exclude_from_sim no)
 		(at 15.875 163.83 0)
